Commit message: 202418

File: ros_industrial_support/urdf/hall/hall.urdf.xacro (robot description, xacro)
@@ -25,4 +25,11 @@
                   izz="${m*(x*x+z*z)/12}" />
 </macro>
+-->
+  <xacro:macro name="box_inertia" params="m x y z">
+    <inertia ixx="${0.0833333 * m * (y*y + z*z)}" ixy="0.0" ixz="0.0"
+      iyy="${0.0833333 * m * (x*x + z*z)}" iyz="0.0"
+      izz="${0.0833333 * m * (x*x + y*y)}" />
+  </xacro:macro>
+<!--
 <macro name="sphere_inertia" params="m r">
         <inertia  ixx="${2*m*r*r/5}" ixy = "0" ixz = "0"
@@ -65,5 +72,5 @@
       <inertial>
         <origin xyz="0 0 0" rpy="0 0 0" />
-        <!--<xacro:box_inertia m="${dummy_mass}" x="${depth}" y="${width}" z="${dummy_thickness}"/>-->
+        <xacro:box_inertia m="${dummy_mass}" x="${depth}" y="${width}" z="${dummy_thickness}"/>
         <mass value="${dummy_mass}" />
       </inertial>
@@ -84,5 +91,5 @@
       <inertial>
         <origin xyz="0 0 0" rpy="0 0 0" />
-        <!--<xacro:box_inertia m="${dummy_mass}" x="${depth}" y="${height}" z="${dummy_thickness}"/>-->
+        <xacro:box_inertia m="${dummy_mass}" x="${depth}" y="${height}" z="${dummy_thickness}"/>
         <mass value="${dummy_mass}" />
       </inertial>
@@ -108,5 +115,5 @@
       <inertial>
         <origin xyz="0 0 0" rpy="0 0 0" />
-        <!--<xacro:box_inertia m="${dummy_mass}" x="${height}" y="${width}" z="${dummy_thickness}"/>-->
+        <xacro:box_inertia m="${dummy_mass}" x="${height}" y="${width}" z="${dummy_thickness}"/>
         <mass value="${dummy_mass}" />
       </inertial>
@@ -132,5 +139,5 @@
       <inertial>
         <origin xyz="0 0 0" rpy="0 0 0" />
-        <!--<xacro:box_inertia m="${dummy_mass}" x="${depth}" y="0.5" z="${dummy_thickness}"/>-->
+        <xacro:box_inertia m="${dummy_mass}" x="${depth}" y="0.5" z="${dummy_thickness}"/>
         <mass value="${dummy_mass}" />
       </inertial>
@@ -156,5 +163,5 @@
       <inertial>
         <origin xyz="0 0 0" rpy="0 0 0" />
-        <!--<xacro:box_inertia m="${dummy_mass}" x="0.5" y="${width}" z="${dummy_thickness}"/>-->
+        <xacro:box_inertia m="${dummy_mass}" x="0.5" y="${width}" z="${dummy_thickness}"/>
         <mass value="${dummy_mass}" />
       </inertial>
